File: PWM/PWM_F24_schemes/PWM_F24.kicad_sch (KiCad schematic)
At the start: 12 parts, among them K1 relay, M1 Motor_DC, Q1 IRL3803, Q2 L78S18CV, U1 Atmega328p-Arduino, U2 IR2110, U3 L7805CV-DG, U4 L7812CV

Commit message: added missing switch to turn on/off the bypass relay
Parts:
- added SW1: SW_Nidec_CAS-120A1, Button_Switch_SMD:Nidec_Copal_CAS-120A, symbol Switch:SW_Nidec_CAS-120A1
Connections:
- net at K1.A2: now also SW1.1 (C); no longer U4.3 (OUT)
- new net: SW1.2 (B), U4.3 (OUT)
Other:
- moved on the sheet: BT1, BT2, M1, U4

Commit message: changed the ATmega 328p chip for the arduino UNO R3.
Parts:
- removed U1: Atmega328p-Arduino, Package_DIP:DIP-28_W7.62mm_LongPads, symbol PCM_SL_Devices:Atmega328p-Arduino
- added A1: Arduino_UNO_R3, Module:Arduino_UNO_R3, symbol MCU_Module:Arduino_UNO_R3
Connections:
- net GND: now also A1.29 (GND)
- net at U2.12 (LIN): now also A1.24 (D9)
- net at U2.9 (VDD), U3.3 (OUT): now also A1.5 (+5V)
Changed lines of the file:
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@@
 	)
 	(junction
-		(at 148.59 24.13)
+		(at 168.91 24.13)
 		(diameter 0)
 		(color 0 0 0 0)
@@
 	(wire
 		(pts
-			(xy 148.59 24.13) (xy 161.29 24.13)
+			(xy 135.89 24.13) (xy 168.91 24.13)
 		)
 		(stroke
@@
 	(wire
 		(pts
-			(xy 148.59 24.13) (xy 148.59 13.97)
-		)
-		(stroke
-			(width 0)
-			(type default)
-		)
-	)
-	(wire
-		(pts
 			(xy 55.88 115.57) (xy 139.7 115.57)
 		)
@@
 	(wire
 		(pts
-			(xy 148.59 13.97) (xy 39.37 13.97)
+			(xy 161.29 87.63) (xy 161.29 83.82)
+		)
+		(stroke
+			(width 0)
+			(type default)
+		)
+	)
+	(wire
+		(pts
+			(xy 39.37 13.97) (xy 168.91 13.97)
 		)
 		(stroke
@@
 	(wire
 		(pts
+			(xy 147.32 68.58) (xy 147.32 63.5)
+		)
+		(stroke
+			(width 0)
+			(type default)
+		)
+	)
+	(wire
+		(pts
 			(xy 139.7 49.53) (xy 138.43 49.53)
 		)
@@
 	(wire
 		(pts
+			(xy 147.32 63.5) (xy 151.13 63.5)
+		)
+		(stroke
+			(width 0)
+			(type default)
+		)
+	)
+	(wire
+		(pts
 			(xy 92.71 52.07) (xy 92.71 46.99)
 		)
@@
 	(wire
 		(pts
-			(xy 135.89 24.13) (xy 148.59 24.13)
+			(xy 168.91 24.13) (xy 168.91 30.48)
 		)
 		(stroke
@@
 	(wire
 		(pts
-			(xy 161.29 24.13) (xy 161.29 30.48)
-		)
-		(stroke
-			(width 0)
-			(type default)
-		)
-	)
-	(wire
-		(pts
 			(xy 138.43 30.48) (xy 135.89 30.48)
 		)
@@
 		(pts
 			(xy 104.14 72.39) (xy 104.14 82.55)
+		)
+		(stroke
+			(width 0)
+			(type default)
+		)
+	)
+	(wire
+		(pts
+			(xy 168.91 13.97) (xy 168.91 24.13)
 		)
 		(stroke
@@
 	)
 	(symbol
-		(lib_id "power:GND")
-		(at 163.83 83.82 0)
+		(lib_id "MCU_Module:Arduino_UNO_R3")
+		(at 163.83 55.88 0)
 		(unit 1)
 		(exclude_from_sim no)
@@
 		(dnp no)
 		(fields_autoplaced yes)
-		(property "Reference" "#PWR04"
-			(at 163.83 90.17 0)
-			(effects
-				(font
-					(size 1.27 1.27)
-				)
-				(hide yes)
-			)
-		)
-		(property "Value" "GND"
-			(at 163.83 88.9 0)
-			(effects
-				(font
-					(size 1.27 1.27)
-				)
-			)
-		)
-		(property "Footprint" ""
-			(at 163.83 83.82 0)
-			(effects
-				(font
-					(size 1.27 1.27)
-				)
-				(hide yes)
-			)
-		)
-		(property "Datasheet" ""
-			(at 163.83 83.82 0)
-			(effects
-				(font
-					(size 1.27 1.27)
-				)
-				(hide yes)
-			)
-		)
-		(property "Description" "Power symbol creates a global label with name \"GND\" , ground"
-			(at 163.83 83.82 0)
-			(effects
-				(font
-					(size 1.27 1.27)
-				)
-				(hide yes)
-			)
+		(property "Reference" "A1"
+			(at 171.1041 27.94 0)
+			(effects
+				(font
+					(size 1.27 1.27)
+				)
+				(justify left)
+			)
+		)
+		(property "Value" "Arduino_UNO_R3"
+			(at 171.1041 30.48 0)
+			(effects
+				(font
+					(size 1.27 1.27)
+				)
+				(justify left)
+			)
+		)
+		(property "Footprint" "Module:Arduino_UNO_R3"
+			(at 163.83 55.88 0)
+			(effects
+				(font
+					(size 1.27 1.27)
+					(italic yes)
+				)
+				(hide yes)
+			)
+		)
+		(property "Datasheet" "https://www.arduino.cc/en/Main/arduinoBoardUno"
+			(at 163.83 55.88 0)
+			(effects
+				(font
+					(size 1.27 1.27)
+				)
+				(hide yes)
+			)
+		)
+		(property "Description" "Arduino UNO Microcontroller Module, release 3"
+			(at 163.83 55.88 0)
+			(effects
+				(font
+					(size 1.27 1.27)
+				)
+				(hide yes)
+			)
+		)
+		(pin "23"
+		)
+		(pin "15"
+		)
+		(pin "11"
+		)
+		(pin "7"
+		)
+		(pin "10"
+		)
+		(pin "13"
+		)
+		(pin "26"
+		)
+		(pin "31"
+		)
+		(pin "4"
+		)
+		(pin "18"
+		)
+		(pin "27"
+		)
+		(pin "17"
+		)
+		(pin "21"
+		)
+		(pin "32"
+		)
+		(pin "25"
+		)
+		(pin "16"
+		)
+		(pin "6"
+		)
+		(pin "12"
+		)
+		(pin "24"
+		)
+		(pin "2"
+		)
+		(pin "29"
+		)
+		(pin "19"
+		)
+		(pin "9"
+		)
+		(pin "5"
+		)
+		(pin "22"
+		)
+		(pin "30"
+		)
+		(pin "20"
+		)
+		(pin "14"
+		)
+		(pin "3"
 		)
 		(pin "1"
+		)
+		(pin "8"
+		)
+		(pin "28"
 		)
 		(instances
 			(project ""
 				(path "/7b5544bd-f439-4d9c-89e6-9bb0e3f4b710"
-					(reference "#PWR04")
+					(reference "A1")
 					(unit 1)
 				)
@@
 	(symbol
 		(lib_id "power:GND")
-		(at 161.29 83.82 0)
+		(at 161.29 87.63 0)
 		(unit 1)
 		(exclude_from_sim no)
@@
 		(fields_autoplaced yes)
 		(property "Reference" "#PWR013"
-			(at 161.29 90.17 0)
+			(at 161.29 93.98 0)
 			(effects
 				(font
@@
 		)
 		(property "Value" "GND"
-			(at 161.29 88.9 0)
+			(at 161.29 92.71 0)
 			(effects
 				(font
@@
 		)
 		(property "Footprint" ""
-			(at 161.29 83.82 0)
+			(at 161.29 87.63 0)
 			(effects
 				(font
@@
 		)
 		(property "Datasheet" ""
-			(at 161.29 83.82 0)
+			(at 161.29 87.63 0)
 			(effects
 				(font
@@
 		)
 		(property "Description" "Power symbol creates a global label with name \"GND\" , ground"
-			(at 161.29 83.82 0)
+			(at 161.29 87.63 0)
 			(effects
 				(font
@@
 					(unit 1)
 				)
-			)
-		)
-	)
-	(symbol
-		(lib_id "PCM_SL_Devices:Atmega328p-Arduino")
-		(at 162.56 58.42 0)
-		(unit 1)
-		(exclude_from_sim no)
-		(in_bom yes)
-		(on_board yes)
-		(dnp no)
-		(fields_autoplaced yes)
-		(property "Reference" "U1"
-			(at 167.2941 27.94 0)
-			(effects
-				(font
-					(size 1.27 1.27)
-				)
-				(justify left)
-			)
-		)
-		(property "Value" "Atmega328p-Arduino"
-			(at 167.2941 30.48 0)
-			(effects
-				(font
-					(size 1.27 1.27)
-				)
-				(justify left)
-			)
-		)
-		(property "Footprint" "Package_DIP:DIP-28_W7.62mm_LongPads"
-			(at 163.83 92.71 0)
-			(effects
-				(font
-					(size 1.27 1.27)
-				)
-				(hide yes)
-			)
-		)
-		(property "Datasheet" ""
-			(at 168.91 90.17 0)
-			(effects
-				(font
-					(size 1.27 1.27)
-				)
-				(hide yes)
-			)
-		)
-		(property "Description" "Atmega328p with Arduino UNO pin mapping(MCU in ArduinoUNO)"
-			(at 162.56 58.42 0)
-			(effects
-				(font
-					(size 1.27 1.27)
-				)
-				(hide yes)
-			)
-		)
-		(pin "1"
-		)
-		(pin "6"
-		)
-		(pin "4"
-		)
-		(pin "11"
-		)
-		(pin "13"
-		)
-		(pin "23"
-		)
-		(pin "15"
-		)
-		(pin "9"
-		)
-		(pin "17"
-		)
-		(pin "3"
-		)
-		(pin "21"
-		)
-		(pin "5"
-		)
-		(pin "16"
-		)
-		(pin "22"
-		)
-		(pin "24"
-		)
-		(pin "12"
-		)
-		(pin "19"
-		)
-		(pin "26"
-		)
-		(pin "28"
-		)
-		(pin "2"
-		)
-		(pin "25"
-		)
-		(pin "8"
-		)
-		(pin "14"
-		)
-		(pin "18"
-		)
-		(pin "20"
-		)
-		(pin "10"
-		)
-		(pin "27"
-		)
-		(pin "7"
-		)
-		(instances
-			(project ""
-				(path "/7b5544bd-f439-4d9c-89e6-9bb0e3f4b710"
-					(reference "U1")
-					(unit 1)
-				)

Commit message: PWM V2.0 Using ESP32 instead of previous Arduino UNO R3
Parts:
- removed A1: Arduino_UNO_R3, Module:Arduino_UNO_R3, symbol MCU_Module:Arduino_UNO_R3
- added A1: ESP32_DevKit_V1_DOIT_36GPIOs, PCM_SL_Development_Boards:DOIT_ESP32_DEVKIT_36Pins, symbol PCM_SL_Development_Board:ESP32_DevKit_V1_DOIT_36GPIOs
- added P1: USB_C_Plug_USB2.0, symbol Connector:USB_C_Plug_USB2.0
- added U5: BOB-12009, BOB-12009:CONV_BOB-12009, symbol BOB-12009:BOB-12009
Connections:
- net GND: now also A1.35 (GND), P1.A1 (GND), P1.A12 (GND), P1.B1 (GND), P1.B12 (GND), U5.GND_1 (GND), U5.GND_2 (GND)
- net at U2.12 (LIN): now also U5.HV1
- net at U2.9 (VDD), U3.3 (OUT): now also U5.HV
- new net: P1.A4 (VBUS), P1.A9 (VBUS), P1.B4 (VBUS), P1.B9 (VBUS)
- new net: A1.36 (VIN), P1.A5 (CC)
- new net: A1.1 (3.3V), U5.LV
- new net: A1.10 (TX2/GPIO16), U5.LV1
Other:
- moved on the sheet: BT1, BT2, BT3, K1, M1, Q1, Q2, R1, SW1, U2, U3, U4

Commit message: PWM V3.0 added function of going in reverse
Parts:
- removed K1: relay, Relay_THT:Relay_SPDT_Fujitsu_FTR-LYCA005x_FormC_Vertical, symbol Relay:Fujitsu_FTR-LYCA005x
- added K2, K3, K4, K5: SPDT, Relay_THT:Relay_SPDT_Fujitsu_FTR-LYCA005x_FormC_Vertical, symbol Relay:Fujitsu_FTR-LYCA005x
Connections:
- net GND: now also K2.12, K2.A1, K3.A1, K4.A1, K5.A1
- net at BT2.1 (+): now also K3.12, K4.12, K5.14; no longer M1.1 (+)
- net at M1.2 (-): now also K2.11
- net at Q1.2 (D): now also K4.14, K5.12
- new net: K2.14, K5.11
- new net: K4.A2, K5.A2
- new net: K3.14, K4.11
- new net: K3.11, M1.1 (+)
- new net: K2.A2, K3.A2
Other:
- moved on the sheet: A1, BT1, BT2, BT3, M1, P1, Q1, Q2, R1, SW1, U2, U3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

Commit message: PWM V3.1 added missing control of relays and added a png image of scheme
Parts:
- added SW2: SW_Nidec_CAS-120A1, Button_Switch_SMD:Nidec_Copal_CAS-120A, symbol Switch:SW_Nidec_CAS-120A1
Connections:
- net at K4.A2, K5.A2: now also SW1.1 (C)
- net at SW1.2 (B), U4.3 (OUT): now also SW2.2 (B)
- net at K2.A2, K3.A2: now also SW2.1 (C)
Other:
- moved on the sheet: SW1
Changed lines of the file:
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@@
 	)
 	(junction
+		(at 58.42 55.88)
+		(diameter 0)
+		(color 0 0 0 0)
+	)
+	(junction
 		(at 24.13 118.11)
 		(diameter 0)
@@
 	)
 	(junction
+		(at 137.16 60.96)
+		(diameter 0)
+		(color 0 0 0 0)
+	)
+	(junction
+		(at 72.39 88.9)
+		(diameter 0)
+		(color 0 0 0 0)
+	)
+	(junction
 		(at 34.29 118.11)
 		(diameter 0)
@@
 	(wire
 		(pts
+			(xy 130.81 82.55) (xy 130.81 88.9)
+		)
+		(stroke
+			(width 0)
+			(type default)
+		)
+	)
+	(wire
+		(pts
 			(xy 143.51 45.72) (xy 140.97 45.72)
 		)
@@
 	(wire
 		(pts
+			(xy 153.67 72.39) (xy 153.67 82.55)
+		)
+		(stroke
+			(width 0)
+			(type default)
+		)
+	)
+	(wire
+		(pts
+			(xy 58.42 49.53) (xy 58.42 55.88)
+		)
+		(stroke
+			(width 0)
+			(type default)
+		)
+	)
+	(wire
+		(pts
 			(xy 24.13 77.47) (xy 24.13 118.11)
 		)
@@
 	(wire
 		(pts
+			(xy 153.67 82.55) (xy 130.81 82.55)
+		)
+		(stroke
+			(width 0)
+			(type default)
+		)
+	)
+	(wire
+		(pts
 			(xy 279.4 156.21) (xy 279.4 33.02)
 		)
@@
 	(wire
 		(pts
-			(xy 153.67 68.58) (xy 153.67 71.12)
+			(xy 41.91 48.26) (xy 52.07 48.26)
 		)
 		(stroke
@@
 	(wire
 		(pts
-			(xy 41.91 48.26) (xy 52.07 48.26)
+			(xy 147.32 52.07) (xy 147.32 38.1)
 		)
 		(stroke
@@
 	(wire
 		(pts
-			(xy 147.32 52.07) (xy 147.32 38.1)
+			(xy 168.91 74.93) (xy 175.26 74.93)
 		)
 		(stroke
@@
 	(wire
 		(pts
-			(xy 168.91 74.93) (xy 175.26 74.93)
+			(xy 147.32 72.39) (xy 153.67 72.39)
 		)
 		(stroke
@@
 	(wire
 		(pts
-			(xy 139.7 68.58) (xy 153.67 68.58)
+			(xy 186.69 83.82) (xy 175.26 83.82)
 		)
 		(stroke
@@
 	(wire
 		(pts
-			(xy 186.69 83.82) (xy 175.26 83.82)
+			(xy 120.65 73.66) (xy 120.65 113.03)
 		)
 		(stroke
@@
 	(wire
 		(pts
-			(xy 120.65 73.66) (xy 120.65 113.03)
+			(xy 132.08 52.07) (xy 137.16 52.07)
 		)
 		(stroke
@@
 	(wire
 		(pts
+			(xy 130.81 88.9) (xy 72.39 88.9)
+		)
+		(stroke
+			(width 0)
+			(type default)
+		)
+	)
+	(wire
+		(pts
 			(xy 81.28 33.02) (xy 147.32 33.02)
 		)
@@
 	(wire
 		(pts
+			(xy 121.92 49.53) (xy 58.42 49.53)
+		)
+		(stroke
+			(width 0)
+			(type default)
+		)
+	)
+	(wire
+		(pts
 			(xy 29.21 110.49) (xy 29.21 132.08)
 		)
@@
 	(wire
 		(pts
-			(xy 129.54 66.04) (xy 129.54 60.96)
+			(xy 137.16 69.85) (xy 137.16 60.96)
 		)
 		(stroke
@@
 	(wire
 		(pts
-			(xy 129.54 60.96) (xy 151.13 60.96)
+			(xy 137.16 60.96) (xy 151.13 60.96)
 		)
 		(stroke
@@
 	(wire
 		(pts
-			(xy 31.75 55.88) (xy 62.23 55.88)
+			(xy 31.75 55.88) (xy 58.42 55.88)
 		)
 		(stroke
@@
 	(wire
 		(pts
+			(xy 137.16 52.07) (xy 137.16 60.96)
+		)
+		(stroke
+			(width 0)
+			(type default)
+		)
+	)
+	(wire
+		(pts
 			(xy 64.77 132.08) (xy 64.77 110.49)
 		)
@@
 	(wire
 		(pts
-			(xy 72.39 86.36) (xy 72.39 95.25)
+			(xy 72.39 86.36) (xy 72.39 88.9)
 		)
 		(stroke
@@
 	(wire
 		(pts
+			(xy 72.39 88.9) (xy 72.39 95.25)
+		)
+		(stroke
+			(width 0)
+			(type default)
+		)
+	)
+	(wire
+		(pts
 			(xy 81.28 73.66) (xy 81.28 33.02)
 		)
@@
 	(wire
 		(pts
+			(xy 58.42 55.88) (xy 62.23 55.88)
+		)
+		(stroke
+			(width 0)
+			(type default)
+		)
+	)
+	(wire
+		(pts
 			(xy 76.2 27.94) (xy 76.2 95.25)
 		)
@@
 	(symbol
 		(lib_id "Switch:SW_Nidec_CAS-120A1")
-		(at 134.62 66.04 0)
+		(at 142.24 69.85 0)
 		(unit 1)
 		(exclude_from_sim no)
@@
 		(fields_autoplaced yes)
 		(property "Reference" "SW1"
-			(at 134.62 57.15 0)
+			(at 142.24 60.96 0)
 			(effects
 				(font
@@
 		)
 		(property "Value" "SW_Nidec_CAS-120A1"
-			(at 134.62 59.69 0)
+			(at 142.24 63.5 0)
 			(effects
 				(font
@@
 		)
 		(property "Footprint" "Button_Switch_SMD:Nidec_Copal_CAS-120A"
-			(at 134.62 76.2 0)
+			(at 142.24 80.01 0)
 			(effects
 				(font
@@
 		)
 		(property "Datasheet" "https://www.nidec-components.com/e/catalog/switch/cas.pdf"
-			(at 134.62 73.66 0)
+			(at 142.24 77.47 0)
 			(effects
 				(font
@@
 		)
 		(property "Description" "Switch, single pole double throw"
-			(at 134.62 66.04 0)
+			(at 142.24 69.85 0)
 			(effects
 				(font
@@
 					(unit 1)
 				)
+			)
+		)
+	)
+	(symbol
+		(lib_id "Switch:SW_Nidec_CAS-120A1")
+		(at 127 52.07 180)
+		(unit 1)
+		(exclude_from_sim no)
+		(in_bom yes)
+		(on_board yes)
+		(dnp no)
+		(fields_autoplaced yes)
+		(property "Reference" "SW2"
+			(at 127 43.18 0)
+			(effects
+				(font
+					(size 1.27 1.27)
+				)
+			)
+		)
+		(property "Value" "SW_Nidec_CAS-120A1"
+			(at 127 45.72 0)
+			(effects
+				(font
+					(size 1.27 1.27)
+				)
+			)
+		)
+		(property "Footprint" "Button_Switch_SMD:Nidec_Copal_CAS-120A"
+			(at 127 41.91 0)
+			(effects
+				(font
+					(size 1.27 1.27)
+				)
+				(hide yes)
+			)
+		)
+		(property "Datasheet" "https://www.nidec-components.com/e/catalog/switch/cas.pdf"
+			(at 127 44.45 0)
+			(effects
+				(font
+					(size 1.27 1.27)
+				)
+				(hide yes)
+			)
+		)
+		(property "Description" "Switch, single pole double throw"
+			(at 127 52.07 0)
+			(effects
+				(font
+					(size 1.27 1.27)
+				)
+				(hide yes)
+			)
+		)
+		(pin "2"
+		)
+		(pin "1"
+		)
+		(pin "3"
+		)
+		(instances
+			(project "PWM_F24"
+				(path "/7b5544bd-f439-4d9c-89e6-9bb0e3f4b710"
+					(reference "SW2")
+					(unit 1)
+				)
